Commit message: Fix XACRO kinematics, CycloneDDS discovery, and joint name consistency
- XACRO: Correct all 6 joint origins (were shifted +1 from original URDF)
  and fix joint limits to match official elephantrobotics values
- CycloneDDS: Remove NetworkInterfaceAddress + AllowMulticast=false from
  cyclonedds_pc.xml; multicast now enabled for local discovery while
  static peer ensures cross-machine unicast to Nano (192.168.0.250)
- Joint names: Update all configs to use official joint2_to_joint1 style
  (mycobot_bridge, moveit_controllers, joint_limits, SRDF, moveit.rviz)
- Arch: Remove joint_rebrander (bridge publishes correct names directly),
  add joint_state_relay (re-stamps Nano timestamps with PC clock),
  remove PushRosNamespace from hw launch (action server at global path),
  set baud=1000000, clean up Dockerfile and dead files

Co-Authored-By: Claude Sonnet 4.6 <noreply@anthropic.com>

File: mycobot_docker/custom_ws/src/mycobot_description/urdf/mycobot_280_jn/mycobot_280_jn.urdf.xacro (robot description, xacro)
@@ -19,27 +19,27 @@
   <link name="link5"><visual><geometry><mesh filename="package://mycobot_description/urdf/mycobot_280_jn/joint6.dae"/></geometry><origin xyz="0 0.00 -0.038" rpy="0 0 0"/></visual></link>
   <link name="link6"><visual><geometry><mesh filename="package://mycobot_description/urdf/mycobot_280_jn/joint7.dae"/></geometry><origin xyz="0.0 0 -0.012" rpy="0 0 0"/><material name="grey"/></visual></link>
-  <joint name="cobot_joint_1" type="revolute">
-    <axis xyz="0 0 1"/><limit effort="100.0" lower="-2.87" upper="2.87" velocity="1.0"/>
-    <parent link="mycobot_base_link"/><child link="link1"/><origin xyz="0 0 0.0706" rpy="0 0 0"/>
+  <joint name="joint2_to_joint1" type="revolute">
+    <axis xyz="0 0 1"/><limit effort="1000.0" lower="-2.9321" upper="2.9321" velocity="3.14"/>
+    <parent link="mycobot_base_link"/><child link="link1"/><origin xyz="0 0 0.15756" rpy="0 0 0"/>
   </joint>
-  <joint name="cobot_joint_2" type="revolute">
-    <axis xyz="0 0 1"/><limit effort="100.0" lower="-2.87" upper="2.87" velocity="1.0"/>
-    <parent link="link1"/><child link="link2"/><origin xyz="0 0 0.15756" rpy="0 0 0"/>
+  <joint name="joint3_to_joint2" type="revolute">
+    <axis xyz="0 0 1"/><limit effort="1000.0" lower="-2.4434" upper="2.4434" velocity="3.14"/>
+    <parent link="link1"/><child link="link2"/><origin xyz="0 0 -0.001" rpy="0 1.5708 -1.5708"/>
   </joint>
-  <joint name="cobot_joint_3" type="revolute">
-    <axis xyz="0 0 1"/><limit effort="100.0" lower="-2.87" upper="2.87" velocity="1.0"/>
-    <parent link="link2"/><child link="link3"/><origin xyz="0 0 -0.001" rpy="0 1.5708 -1.5708"/>
+  <joint name="joint4_to_joint3" type="revolute">
+    <axis xyz="0 0 1"/><limit effort="1000.0" lower="-2.6179" upper="2.6179" velocity="3.14"/>
+    <parent link="link2"/><child link="link3"/><origin xyz="-0.1104 0 0" rpy="0 0 0"/>
   </joint>
-  <joint name="cobot_joint_4" type="revolute">
-    <axis xyz="0 0 1"/><limit effort="100.0" lower="-2.87" upper="2.87" velocity="1.0"/>
-    <parent link="link3"/><child link="link4"/><origin xyz="-0.1104 0 0" rpy="0 0 0"/>
+  <joint name="joint5_to_joint4" type="revolute">
+    <axis xyz="0 0 1"/><limit effort="1000.0" lower="-2.6179" upper="2.6179" velocity="3.14"/>
+    <parent link="link3"/><child link="link4"/><origin xyz="-0.096 0 0.06462" rpy="0 0 -1.5708"/>
   </joint>
-  <joint name="cobot_joint_5" type="revolute">
-    <axis xyz="0 0 1"/><limit effort="100.0" lower="-2.87" upper="2.87" velocity="1.0"/>
-    <parent link="link4"/><child link="link5"/><origin xyz="-0.096 0 0.06462" rpy="0 0 -1.5708"/>
+  <joint name="joint6_to_joint5" type="revolute">
+    <axis xyz="0 0 1"/><limit effort="1000.0" lower="-2.7052" upper="2.7925" velocity="3.14"/>
+    <parent link="link4"/><child link="link5"/><origin xyz="0 -0.07318 0" rpy="1.5708 -1.5708 0"/>
   </joint>
-  <joint name="cobot_joint_6" type="revolute">
-    <axis xyz="0 0 1"/><limit effort="100.0" lower="-3.05" upper="3.05" velocity="1.0"/>
-    <parent link="link5"/><child link="link6"/><origin xyz="0 -0.07318 0" rpy="1.5708 -1.5708 0"/>
+  <joint name="joint6output_to_joint6" type="revolute">
+    <axis xyz="0 0 1"/><limit effort="1000.0" lower="-3.14159" upper="3.14159" velocity="3.14"/>
+    <parent link="link5"/><child link="link6"/><origin xyz="0 0.0456 0" rpy="-1.5708 0 0"/>
   </joint>
 </robot>

Commit message: Fix RViz SIGABRT: add collision geometry to URDF links 1-6
moveit_rviz_plugin in Galactic has a heap corruption bug (munmap_chunk:
invalid pointer) when loading robot models where links have visual
geometry but no collision geometry. Adding collision elements (same
mesh as visual) fixes it. This is the root cause of all the SIGSEGV/-11
and SIGABRT/-6 crashes since RViz started crashing.

Also restore Query Goal State: true in moveit.rviz (interactive goal
marker was disabled during crash investigation).

Co-Authored-By: Claude Sonnet 4.6 <noreply@anthropic.com>

File: mycobot_docker/custom_ws/src/mycobot_description/urdf/mycobot_280_jn/mycobot_280_jn.urdf.xacro (robot description, xacro)
@@ -13,10 +13,28 @@
     </collision>
   </link>
-  <link name="link1"><visual><geometry><mesh filename="package://mycobot_description/urdf/mycobot_280_jn/joint2.dae"/></geometry><origin xyz="0.0 0 -0.06096" rpy="0 0 -1.5708"/></visual></link>
-  <link name="link2"><visual><geometry><mesh filename="package://mycobot_description/urdf/mycobot_280_jn/joint3.dae"/></geometry><origin xyz="0.0 0 0.03256" rpy="0 -1.5708 0"/></visual></link>
-  <link name="link3"><visual><geometry><mesh filename="package://mycobot_description/urdf/mycobot_280_jn/joint4.dae"/></geometry><origin xyz="0.0 0 0.03056" rpy="0 -1.5708 0"/></visual></link>
-  <link name="link4"><visual><geometry><mesh filename="package://mycobot_description/urdf/mycobot_280_jn/joint5.dae"/></geometry><origin xyz="0.0 0 -0.03356" rpy="0 -1.5708 1.5708"/></visual></link>
-  <link name="link5"><visual><geometry><mesh filename="package://mycobot_description/urdf/mycobot_280_jn/joint6.dae"/></geometry><origin xyz="0 0.00 -0.038" rpy="0 0 0"/></visual></link>
-  <link name="link6"><visual><geometry><mesh filename="package://mycobot_description/urdf/mycobot_280_jn/joint7.dae"/></geometry><origin xyz="0.0 0 -0.012" rpy="0 0 0"/><material name="grey"/></visual></link>
+  <link name="link1">
+    <visual><geometry><mesh filename="package://mycobot_description/urdf/mycobot_280_jn/joint2.dae"/></geometry><origin xyz="0.0 0 -0.06096" rpy="0 0 -1.5708"/></visual>
+    <collision><geometry><mesh filename="package://mycobot_description/urdf/mycobot_280_jn/joint2.dae"/></geometry><origin xyz="0.0 0 -0.06096" rpy="0 0 -1.5708"/></collision>
+  </link>
+  <link name="link2">
+    <visual><geometry><mesh filename="package://mycobot_description/urdf/mycobot_280_jn/joint3.dae"/></geometry><origin xyz="0.0 0 0.03256" rpy="0 -1.5708 0"/></visual>
+    <collision><geometry><mesh filename="package://mycobot_description/urdf/mycobot_280_jn/joint3.dae"/></geometry><origin xyz="0.0 0 0.03256" rpy="0 -1.5708 0"/></collision>
+  </link>
+  <link name="link3">
+    <visual><geometry><mesh filename="package://mycobot_description/urdf/mycobot_280_jn/joint4.dae"/></geometry><origin xyz="0.0 0 0.03056" rpy="0 -1.5708 0"/></visual>
+    <collision><geometry><mesh filename="package://mycobot_description/urdf/mycobot_280_jn/joint4.dae"/></geometry><origin xyz="0.0 0 0.03056" rpy="0 -1.5708 0"/></collision>
+  </link>
+  <link name="link4">
+    <visual><geometry><mesh filename="package://mycobot_description/urdf/mycobot_280_jn/joint5.dae"/></geometry><origin xyz="0.0 0 -0.03356" rpy="0 -1.5708 1.5708"/></visual>
+    <collision><geometry><mesh filename="package://mycobot_description/urdf/mycobot_280_jn/joint5.dae"/></geometry><origin xyz="0.0 0 -0.03356" rpy="0 -1.5708 1.5708"/></collision>
+  </link>
+  <link name="link5">
+    <visual><geometry><mesh filename="package://mycobot_description/urdf/mycobot_280_jn/joint6.dae"/></geometry><origin xyz="0 0.00 -0.038" rpy="0 0 0"/></visual>
+    <collision><geometry><mesh filename="package://mycobot_description/urdf/mycobot_280_jn/joint6.dae"/></geometry><origin xyz="0 0.00 -0.038" rpy="0 0 0"/></collision>
+  </link>
+  <link name="link6">
+    <visual><geometry><mesh filename="package://mycobot_description/urdf/mycobot_280_jn/joint7.dae"/></geometry><origin xyz="0.0 0 -0.012" rpy="0 0 0"/><material name="grey"/></visual>
+    <collision><geometry><mesh filename="package://mycobot_description/urdf/mycobot_280_jn/joint7.dae"/></geometry><origin xyz="0.0 0 -0.012" rpy="0 0 0"/></collision>
+  </link>
   <joint name="joint2_to_joint1" type="revolute">
     <axis xyz="0 0 1"/><limit effort="1000.0" lower="-2.9321" upper="2.9321" velocity="3.14"/>
