Commit message: Add camera module v2.0 ao modelo + pose de observacao no modo visao
- URDF: camera_link (caixa 64x16x36mm + lente) no topo do corpo da
  pump, olhando na direcao do copo (+y do link6); camera_optical no
  padrao ROS (z sai da lente). Offsets aproximados — calibrar no real.
- pick_and_place --scan-pose <nome>: no modo visao o braco vai antes
  para a pose de observacao (grave com SAVE_POSE.sh scan) e so entao
  espera a deteccao YOLO
- RUN_MOCK_PC.sh: colcon build automatico dos 3 pacotes no arranque

File: mycobot_docker/custom_ws/src/mycobot_description/urdf/mycobot_280_jn/mycobot_280_jn.urdf.xacro (robot description, xacro)
@@ -49,4 +49,22 @@
   <!-- suction cup tip frame (TCP) -->
   <link name="pump_tcp"/>
+  <!-- USB camera module v2.0 (myCobot_cameraHolder_J6), eye-in-hand.
+       Sem mesh oficial: caixa 64x16x36mm + lente. Montada no topo do
+       corpo da pump, olhando na MESMA direção do copo (+y do link6) —
+       quando o copo aponta p/ baixo, a câmera vê a mesa/lata.
+       POSIÇÃO APROXIMADA: ajustar os offsets após montar no robô real
+       (calibração câmera-flange). -->
+  <link name="camera_link">
+    <visual>
+      <geometry><box size="0.064 0.016 0.036"/></geometry>
+      <origin xyz="0 0 0" rpy="0 0 0"/>
+      <material name="white"/>
+    </visual>
+    <visual>
+      <geometry><cylinder radius="0.007" length="0.006"/></geometry>
+      <origin xyz="0 0.010 0" rpy="1.5708 0 0"/>
+      <material name="grey"/>
+    </visual>
+  </link>
   <joint name="joint2_to_joint1" type="revolute">
     <axis xyz="0 0 1"/><limit effort="1000.0" lower="-2.9321" upper="2.9321" velocity="3.14"/>
@@ -93,3 +111,15 @@
     <origin xyz="0 0.0037 -0.0145" rpy="3.14159 0 0"/>
   </joint>
+  <!-- Câmera no topo do corpo da pump (acima dos 73mm do corpo) -->
+  <joint name="link6_to_camera" type="fixed">
+    <parent link="link6"/><child link="camera_link"/>
+    <origin xyz="0 -0.002 0.09" rpy="0 0 0"/>
+  </joint>
+  <!-- Frame óptico (convenção ROS: z sai da lente, x direita, y baixo).
+       z óptico = +y do link6 = direção do copo de sucção. -->
+  <link name="camera_optical"/>
+  <joint name="camera_to_optical" type="fixed">
+    <parent link="camera_link"/><child link="camera_optical"/>
+    <origin xyz="0 0.013 0" rpy="-1.5708 0 0"/>
+  </joint>
 </robot>

Commit message: Substitui camera improvisada pelo camera_flange oficial (AI Kit)
- camera_flange.dae oficial (mycobot_ros/noetic, 280 JN) montada entre
  o flange e a pump, com os transforms do modelo combinado oficial
  mycobot_280m5_with_camera_flange_pump.urdf:
  link6 -> camera_flange (0 0 0.01, rpy 1.579 0 0)
  camera_flange -> pump_head (0 0 0.01, rpy -1.579 0 0)
- pump_head com origens oficiais do combinado (0, 0.008, 0.009,
  rpy 1.5708 0 0); pump_tcp recalculado por FK: copo em
  (0, 0.02245, 0.02066) no pump_head = (0, 0.0125, 0.0306) no link6
- colisao da camera_flange por box primitiva (mesh em mm, bug assimp)
- camera_optical no centro da placa olhando na direcao do copo
  (calibrar offsets no robo real)
- SRDF: pares camera_flange (link6/pump_head Adjacent, link5 Never)

File: mycobot_docker/custom_ws/src/mycobot_description/urdf/mycobot_280_jn/mycobot_280_jn.urdf.xacro (robot description, xacro)
@@ -35,8 +35,23 @@
     </collision>
   </link>
+  <!-- Camera flange oficial (AI Kit): monta ENTRE o flange e a pump.
+       Mesh oficial mycobot_ros/noetic (COLLADA em mm → colisão por box
+       primitiva, bbox 83x9x34.5mm). -->
+  <link name="camera_flange">
+    <visual>
+      <geometry><mesh filename="package://mycobot_description/urdf/mycobot_280_jn/camera_flange.dae"/></geometry>
+      <origin xyz="0.024 -0.008 0.0" rpy="0 3.14159 0"/>
+    </visual>
+    <collision>
+      <geometry><box size="0.083 0.009 0.0345"/></geometry>
+      <origin xyz="0.024 -0.0045 -0.0005" rpy="0 3.14159 0"/>
+    </collision>
+  </link>
   <link name="pump_head">
+    <!-- Origens do modelo oficial COMBINADO camera_flange + pump
+         (mycobot_280m5_with_camera_flange_pump.urdf) -->
     <visual>
       <geometry><mesh filename="package://mycobot_description/urdf/mycobot_280_jn/pump_head.dae"/></geometry>
-      <origin xyz="0.0 -0.008 0.0" rpy="0 0 0"/>
+      <origin xyz="0.0 0.008 0.009" rpy="1.5708 0 0"/>
     </visual>
     <!-- Colisão: caixa primitiva (bbox do mesh, 24.5x63x26.7mm), mesmo
@@ -44,27 +59,9 @@
     <collision>
       <geometry><box size="0.0245 0.063 0.0267"/></geometry>
-      <origin xyz="0.0 0.0235 -0.0011" rpy="0 0 0"/>
+      <origin xyz="0.0 0.0091 0.0405" rpy="1.5708 0 0"/>
     </collision>
   </link>
   <!-- suction cup tip frame (TCP) -->
   <link name="pump_tcp"/>
-  <!-- USB camera module v2.0 (myCobot_cameraHolder_J6), eye-in-hand.
-       Sem mesh oficial: caixa 64x16x36mm + lente. Montada no topo do
-       corpo da pump, olhando na MESMA direção do copo (+y do link6) —
-       quando o copo aponta p/ baixo, a câmera vê a mesa/lata.
-       POSIÇÃO APROXIMADA: ajustar os offsets após montar no robô real
-       (calibração câmera-flange). -->
-  <link name="camera_link">
-    <visual>
-      <geometry><box size="0.064 0.016 0.036"/></geometry>
-      <origin xyz="0 0 0" rpy="0 0 0"/>
-      <material name="white"/>
-    </visual>
-    <visual>
-      <geometry><cylinder radius="0.007" length="0.006"/></geometry>
-      <origin xyz="0 0.010 0" rpy="1.5708 0 0"/>
-      <material name="grey"/>
-    </visual>
-  </link>
   <joint name="joint2_to_joint1" type="revolute">
     <axis xyz="0 0 1"/><limit effort="1000.0" lower="-2.9321" upper="2.9321" velocity="3.14"/>
@@ -96,30 +93,31 @@
     <origin xyz="0 0 0" rpy="0 0 0"/>
   </joint>
-  <!-- Pump head (suction nozzle) at the end effector -->
-  <joint name="link6_to_pump_head" type="fixed">
-    <parent link="link6"/><child link="pump_head"/>
+  <!-- Camera flange no flange do link6 (transform oficial) -->
+  <joint name="link6_to_camera_flange" type="fixed">
+    <parent link="link6"/><child link="camera_flange"/>
     <origin xyz="0 0 0.01" rpy="1.579 0 0"/>
   </joint>
-  <!-- TCP at the suction cup face.
-       Mesh analysis (pump_head.dae, mm): cup = Ø20mm ring at (0, 11.66, -14.45),
-       facing -z of the mesh. Visual origin shifts y by -8mm, so in the
-       pump_head frame the cup face is at (0, 0.0037, -0.0145).
-       rpy="pi 0 0" flips z so pump_tcp z points OUT of the cup (into the
-       object being sucked) — in link6 frame that is the +y direction. -->
+  <!-- Pump pendurada NA camera flange (transform oficial do combinado) -->
+  <joint name="camera_flange_to_pump_head" type="fixed">
+    <parent link="camera_flange"/><child link="pump_head"/>
+    <origin xyz="0 0 0.01" rpy="-1.579 0 0"/>
+  </joint>
+  <!-- TCP na face do copo de sucção.
+       Mesh (mm): anel Ø20 em (0, 11.66, -14.45) olhando -z do mesh.
+       Com a origem visual oficial (0, 0.008, 0.009, rpy 1.5708 0 0),
+       o copo fica em (0, 0.02245, 0.02066) no frame pump_head, sucção
+       para +y_ph. rpy=(-pi/2,0,0) põe o z do TCP saindo do copo —
+       no link6 isso é +y (FK verificado: copo em (0, 0.0125, 0.0306)). -->
   <joint name="pump_head_to_tcp" type="fixed">
     <parent link="pump_head"/><child link="pump_tcp"/>
-    <origin xyz="0 0.0037 -0.0145" rpy="3.14159 0 0"/>
+    <origin xyz="0 0.02245 0.02066" rpy="-1.5708 0 0"/>
   </joint>
-  <!-- Câmera no topo do corpo da pump (acima dos 73mm do corpo) -->
-  <joint name="link6_to_camera" type="fixed">
-    <parent link="link6"/><child link="camera_link"/>
-    <origin xyz="0 -0.002 0.09" rpy="0 0 0"/>
-  </joint>
-  <!-- Frame óptico (convenção ROS: z sai da lente, x direita, y baixo).
-       z óptico = +y do link6 = direção do copo de sucção. -->
+  <!-- Frame óptico da câmera (convenção ROS: z sai da lente).
+       A câmera do flange olha na direção do copo (-z da camera_flange).
+       Posição aproximada no centro da placa — CALIBRAR no robô real. -->
   <link name="camera_optical"/>
-  <joint name="camera_to_optical" type="fixed">
-    <parent link="camera_link"/><child link="camera_optical"/>
-    <origin xyz="0 0.013 0" rpy="-1.5708 0 0"/>
+  <joint name="camera_flange_to_optical" type="fixed">
+    <parent link="camera_flange"/><child link="camera_optical"/>
+    <origin xyz="0.024 -0.0045 -0.017" rpy="3.14159 0 0"/>
   </joint>
 </robot>
